Commit message: Fixing name problems

File: urdf/blueboat.xacro (robot description, xacro)
@@ -19,5 +19,5 @@
         <origin rpy="3.1416 0 -1.5708" xyz="0 0 0"/>
         <geometry>
-          <mesh filename="package://blueboat_stonefish/meshes/blueboat.dae" scale="1 1 1"/>
+          <mesh filename="package://blueboat_stonefish_core/meshes/blueboat.dae" scale="1 1 1"/>
         </geometry>
         <material name="blue"><color rgba="0 0 1 1"/></material>

Commit message: Some lauch changes

File: urdf/blueboat.xacro (robot description, xacro)
@@ -26,5 +26,5 @@
         <origin rpy="3.1416 0 -1.5708" xyz="0 0 0"/>
         <geometry>
-          <mesh filename="package://blueboat_stonefish/meshes/blueboat.dae" scale="1 1 1"/>
+          <mesh filename="package://blueboat_stonefish_core/meshes/blueboat.dae" scale="1 1 1"/>
         </geometry>
       </collision>
